File: v86p-ide.kicad_pcb (KiCad board)
At the start: 2 copper layers, 152.8 x 50 mm, 61 parts, among them J1 Conn_02x20_Odd_Even, J2 Conn_01x02, J3 Conn_02x20_Odd_Even, J4 Conn_01x03, J5 Conn_02x04_Odd_Even, J6 Conn_01x01, U1 74LS573, U10 74LS688, U11 74LS245, U12 74AHC1G04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

Commit message: Fixed DRC errors
Parts:
- moved R16 2.50 mm to (64.8, 66.0)
- moved R18 2.50 mm to (62.3, 66.0)
- moved R1 0.30 mm to (201.5, 41.2)
Routing:
- net (no net): track 1.81 -> 0.00 mm
- net Net-(D1-Pad1): track 1.84 -> 2.34 mm
